Commit message: switch to odrive

File: ros_ws/src/mirobot_description/urdf/macros.xacro (robot description, xacro)
@@ -73,5 +73,5 @@
       <material>Gazebo/FlatBlack</material>
     </gazebo>
-    <joint name="${lr}_wheel_hinge" type="continuous">
+    <joint name="wheel_${lr}_joint" type="continuous">
       <parent link="chassis"/>
       <child link="${lr}_wheel"/>
@@ -90,9 +90,9 @@
     <transmission name="${lr}_trans">
       <type>transmission_interface/SimpleTransmission</type>
-      <joint name="${lr}_wheel_hinge">
-        <hardwareInterface>hardware_interface/EffortJointInterface</hardwareInterface>
+      <joint name="wheel_${lr}_joint">
+        <hardwareInterface>hardware_interface/VelocityJointInterface</hardwareInterface>
       </joint>
       <actuator name="${lr}Motor">
-        <hardwareInterface>hardware_interface/EffortJointInterface</hardwareInterface>
+        <hardwareInterface>hardware_interface/VelocityJointInterface</hardwareInterface>
         <mechanicalReduction>10</mechanicalReduction>
         <!--mechanicalReduction>1</mechanicalReduction-->

File: ros_ws/src/mirobot_description/urdf/mirobot.xacro (robot description, xacro)
@@ -78,6 +78,6 @@
 		</inertial>
 	</link>
-	<wheel lr="left" tY="-1"/>
-	<wheel lr="right" tY="1"/>
+	<wheel lr="0" tY="-1"/>
+	<wheel lr="1" tY="1"/>
 	<!-- Sensor models -->
 	<xacro:include filename="$(find mirobot_description)/urdf/sensors.xacro" />

File: ros_ws/src/mirobot_description/urdf/mirobot_properties.xacro (robot description, xacro)
@@ -5,31 +5,31 @@
 	<!-- Chassis properties -->
 	<xacro:property name="chassisHeight" value="0.1"/>
-	<xacro:property name="chassisLength" value="0.225"/>
-	<xacro:property name="chassisWidth" value="0.165"/>
+	<xacro:property name="chassisLength" value="0.44"/>
+	<xacro:property name="chassisWidth" value="0.465"/>
 	<xacro:property name="chassisMass" value="2.0"/>
 	<!-- Caster wheel properties -->
 	<xacro:property name="casterRadius" value="0.021"/>
 	<xacro:property name="casterMass" value="0.09"/>
-	<xacro:property name="casterOffsetX" value="0.091"/>
+	<xacro:property name="casterOffsetX" value="0.232"/>
 	<!-- Differential-drive wheels properties -->
-	<xacro:property name="wheelWidth" value="0.06"/>
-	<xacro:property name="wheelRadius" value="0.065"/>
-	<xacro:property name="wheelMass" value="0.185"/>
-	<xacro:property name="wheelOffsetY" value="0.130"/>
+	<xacro:property name="wheelWidth" value="0.05"/>
+	<xacro:property name="wheelRadius" value="0.085"/>
+	<xacro:property name="wheelMass" value="1"/>
+	<xacro:property name="wheelOffsetY" value="0.105"/>
 	<!-- Hokuyo laser properties -->
 	<xacro:property name="hokuyoMass" value="0.01"/>
 	<xacro:property name="hokuyoLength" value="0.05"/>
 	<xacro:property name="hokuyoWidth" value="0.05"/>
-	<xacro:property name="hokuyoHeight" value="0.07"/>
-	<xacro:property name="hokuyoOffsetX" value="0.035"/>
+	<xacro:property name="hokuyoHeight" value="0.055"/>
+	<xacro:property name="hokuyoOffsetX" value="0.232"/>
 	<!--xacro:property name="hokuyoOffsetX" value="0.05"/-->
-	<xacro:property name="hokuyoOffsetZ" value="0.1135"/>
+	<xacro:property name="hokuyoOffsetZ" value="0.025"/>
 	<!--xacro:property name="hokuyoOffsetZ" value="0.1125"/-->
 	<!-- Camera properties -->
-	<xacro:property name="cameraLength" value="0.04"/>
-	<xacro:property name="cameraWidth" value="0.08"/>
-	<xacro:property name="cameraHeight" value="0.03"/>
+	<xacro:property name="cameraLength" value="0.11"/>
+	<xacro:property name="cameraWidth" value="0.002"/>
+	<xacro:property name="cameraHeight" value="0.035"/>
 	<xacro:property name="cameraMass" value="0.01"/>
-	<xacro:property name="cameraOffsetX" value="0.095"/>
-	<xacro:property name="cameraOffsetZ" value="0.06"/>
+	<xacro:property name="cameraOffsetX" value="0.232"/>
+	<xacro:property name="cameraOffsetZ" value="0.025"/>
 </robot>
