Commit message: clean up nav config, experiment with rtabmap

File: ros_ws/src/mirobot_description/urdf/MiroBot.urdf (robot description, URDF)
Before this commit: robot MiroBot, 7 links, 6 joints
Links:
- link base_link: mass 0.002 -> None
- link camera_link: mass 0.001 -> None
- link l_caster_wheel_link: mass 0.001 -> None
- link l_wheel_link: mass 0.001 -> None
- link lidar_link: mass 0.001 -> None
- link r_caster_wheel_link: mass 0.001 -> None
- link r_wheel_link: mass 0.001 -> None

Commit message: initial push

File: ros_ws/src/mirobot_description/urdf/MiroBot.urdf (robot description, URDF)
Before this commit: robot MiroBot, 7 links, 6 joints
Links:
- removed link camera_link
- removed link lidar_link
- added link d400_link; visual mesh filename=package://mirobot_description/meshes/d435.dae
- added link laser_link; visual mesh filename=package://mirobot_description/meshes/lidar.dae
- added link t265_link; visual mesh filename=package://mirobot_description/meshes/t265.dae
- link base_link: geometry collision box size=0.42 0.42 0.42; visual mesh filename=package://mirobot_description/meshes/base.dae
Joints:
- removed joint camera_joint
- removed joint lidar_joint
- added joint d400_joint: type fixed, parent base_link, child d400_link, origin xyz=0.300 0 0.2 rpy=0 0 0
- added joint laser_joint: type fixed, parent base_link, child laser_link, origin xyz=0.22 0 0.001 rpy=3.141527 0 0
- added joint t265_joint: type fixed, parent base_link, child t265_link, origin xyz=0.305 0 0.225 rpy=0 0 0
- joint l_wheel_joint: axis 1 0 0 -> 0 1 0; origin xyz=0 0.26 0 rpy=0 0 0 -> xyz=0 0.135 0 rpy=0 0 0
- joint r_wheel_joint: axis 1 0 0 -> 0 1 0; origin xyz=0 -0.26 0 rpy=3.141527 0 0 -> xyz=0 -0.135 0 rpy=3.141527 0 0

Commit message: reconfigure nav stack

File: ros_ws/src/mirobot_description/urdf/MiroBot.urdf (robot description, URDF)
Before this commit: robot MiroBot, 8 links, 7 joints
Links:
- removed link d400_link
- removed link t265_link
Joints:
- removed joint d400_joint
- removed joint t265_joint
