Commit message: add bumper sensor in gazebo

File: ros_ws/src/qb_description/urdf/qb.xacro (robot description, xacro)
@@ -119,8 +119,10 @@
     <material name="silver"/>
   </visual>
-  <collision>
-    <origin rpy="0 0 0" xyz="-0.310634 -0.0 -0.3272"/>
-    <geometry>
-      <mesh filename="package://qb_description/meshes/t265_link.stl" scale="0.001 0.001 0.001"/>
+  <collision name="t265_collision_box">
+    <origin rpy="0 0 0" xyz="0.03 -0.0 -0.2"/>
+    <!--<origin rpy="0 0 0" xyz="-0.310634 -0.0 -0.3272"/>-->
+    <geometry>
+      <box size="0.03 0.4 0.05"/>
+      <!--<mesh filename="package://qb_description/meshes/t265_link.stl" scale="0.001 0.001 0.001"/>-->
     </geometry>
   </collision>

Commit message: update packages to work with ROS noetic

File: ros_ws/src/qb_description/urdf/qb.xacro (robot description, xacro)
@@ -201,5 +201,5 @@
 </joint>
 <joint name="lidar_joint" type="fixed">
-  <origin rpy="0 0 0" xyz="0.23 0.0 0.065"/>
+  <origin rpy="3.141592 0 0" xyz="0.23 0.0 0.065"/>
   <parent link="base_link"/>
   <child link="laser_link"/>

Commit message: add ira_laser_tools and aruco localiser repos.

File: ros_ws/src/qb_description/urdf/qb.xacro (robot description, xacro)
@@ -196,5 +196,5 @@
 </joint>
 <joint name="d435_joint" type="fixed">
-  <origin rpy="0 0 0" xyz="-0.135 0.0 0.3025"/>
+  <origin rpy="0 0 3.141592" xyz="-0.135 0.0 0.3025"/>
   <parent link="base_link"/>
   <child link="d435_link"/>
